File: hardware/Shield.brd (EAGLE design)
At the start: 53.3 x 55.9 mm, 25 parts, among them J1 AVR_SPI_PRG_6PTH, Q8 TIP120, U2 LM78XX-TO252-3, U4 ATMEGA328P_PDIP, Y1 16Mhz

Commit message: Switched wiring for lights to clean up board layout
Connections:
- net N$2: now also LIGHT.8; no longer LIGHT.1
- net N$3: now also LIGHT.6; no longer LIGHT.3
- net N$4: now also LIGHT.4; no longer LIGHT.5
- net N$5: now also LIGHT.2; no longer LIGHT.7
- net VCC: now also LIGHT.1, LIGHT.3, LIGHT.5, LIGHT.7; no longer LIGHT.2, LIGHT.4, LIGHT.6, LIGHT.8
Routing:
- net VCC: track 140.2 -> 124.0 mm
- net N$5: track 30.7 -> 15.1 mm
- net N$4: track 26.0 -> 16.0 mm
- net N$2: track 13.6 -> 18.5 mm
- net N$3: track 21.3 -> 17.2 mm
Other:
- board text added: "UCI Gate v3.1"
- board text removed: "UCI Gate v3.0.1"
Changed lines of the file:
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@@
 <wire x1="53.34" y1="55.88" x2="0" y2="55.88" width="0" layer="20"/>
 <wire x1="0" y1="55.88" x2="0" y2="0" width="0" layer="20"/>
-<text x="37.465" y="52.07" size="1.778" layer="22" rot="MR0">UCI Gate v3.0.1</text>
+<text x="37.465" y="52.07" size="1.778" layer="22" rot="MR0">UCI Gate v3.1</text>
 <text x="30.48" y="0" size="1.778" layer="21">- +</text>
 <text x="23.495" y="0" size="1.778" layer="21">- +</text>
@@
 <contactref element="C6" pad="1"/>
 <contactref element="PWR" pad="1"/>
-<contactref element="LIGHT" pad="2"/>
-<contactref element="LIGHT" pad="4"/>
-<contactref element="LIGHT" pad="8"/>
-<contactref element="LIGHT" pad="6"/>
 <contactref element="U$1" pad="9"/>
 <contactref element="GATE" pad="1"/>
 <contactref element="C8" pad="1"/>
 <contactref element="U2" pad="1"/>
-<wire x1="41.275" y1="12.065" x2="41.275" y2="17.78" width="0.6096" layer="1"/>
 <wire x1="6.35" y1="5.08" x2="6.35" y2="3.81" width="0.6096" layer="16"/>
 <wire x1="6.35" y1="3.81" x2="8.89" y2="1.27" width="0.6096" layer="16"/>
@@
 <wire x1="15.24" y1="1.27" x2="21.59" y2="1.27" width="0.6096" layer="16"/>
 <wire x1="21.59" y1="1.27" x2="34.925" y2="1.27" width="0.6096" layer="16"/>
-<wire x1="34.925" y1="1.27" x2="36.195" y2="2.54" width="0.6096" layer="16"/>
-<wire x1="36.195" y1="2.54" x2="36.195" y2="5.08" width="0.6096" layer="16"/>
-<wire x1="36.195" y1="5.08" x2="37.465" y2="6.35" width="0.6096" layer="16"/>
-<wire x1="37.465" y1="6.35" x2="48.26" y2="6.35" width="0.6096" layer="16"/>
-<wire x1="48.26" y1="6.35" x2="49.53" y2="7.62" width="0.6096" layer="16"/>
-<wire x1="49.53" y1="7.62" x2="49.53" y2="11.43" width="0.6096" layer="16"/>
-<wire x1="49.53" y1="11.43" x2="48.895" y2="12.065" width="0.6096" layer="16"/>
 <wire x1="13.335" y1="5.08" x2="13.335" y2="3.175" width="0.6096" layer="16"/>
 <wire x1="13.335" y1="3.175" x2="15.24" y2="1.27" width="0.6096" layer="16"/>
 <wire x1="20.32" y1="5.08" x2="20.32" y2="2.54" width="0.6096" layer="16"/>
 <wire x1="20.32" y1="2.54" x2="21.59" y2="1.27" width="0.6096" layer="16"/>
-<wire x1="48.895" y1="12.065" x2="46.355" y2="12.065" width="0.6096" layer="1"/>
-<wire x1="46.355" y1="12.065" x2="43.815" y2="12.065" width="0.6096" layer="1"/>
-<wire x1="43.815" y1="12.065" x2="41.275" y2="12.065" width="0.6096" layer="1"/>
 <wire x1="1.27" y1="43.18" x2="1.905" y2="43.815" width="0.6096" layer="1"/>
 <wire x1="1.905" y1="43.815" x2="2.4384" y2="43.815" width="0.6096" layer="1"/>
 <wire x1="2.4384" y1="43.815" x2="2.794" y2="44.1706" width="0.6096" layer="1"/>
-<wire x1="26.67" y1="21.33" x2="26.67" y2="22.86" width="0.6096" layer="1"/>
-<wire x1="26.67" y1="22.86" x2="27.305" y2="23.495" width="0.6096" layer="1"/>
-<wire x1="27.305" y1="23.495" x2="35.56" y2="23.495" width="0.6096" layer="1"/>
-<wire x1="35.56" y1="23.495" x2="41.275" y2="17.78" width="0.6096" layer="1"/>
 <wire x1="6.35" y1="24.13" x2="6.35" y2="25.4" width="0.6096" layer="1"/>
 <wire x1="6.35" y1="25.4" x2="5.08" y2="26.67" width="0.6096" layer="1"/>
@@
 <wire x1="8.215" y1="19.725" x2="6.35" y2="21.59" width="0.6096" layer="1"/>
 <wire x1="6.35" y1="21.59" x2="6.35" y2="24.13" width="0.6096" layer="1"/>
+<contactref element="LIGHT" pad="7"/>
+<contactref element="LIGHT" pad="5"/>
+<contactref element="LIGHT" pad="3"/>
+<contactref element="LIGHT" pad="1"/>
+<wire x1="34.925" y1="1.27" x2="36.195" y2="2.54" width="0.6096" layer="16"/>
+<wire x1="36.195" y1="2.54" x2="36.195" y2="5.08" width="0.6096" layer="16"/>
+<wire x1="36.195" y1="5.08" x2="40.005" y2="8.89" width="0.6096" layer="16"/>
+<wire x1="40.005" y1="8.89" x2="40.005" y2="9.525" width="0.6096" layer="16"/>
+<wire x1="40.005" y1="9.525" x2="42.545" y2="9.525" width="0.6096" layer="16"/>
+<wire x1="42.545" y1="9.525" x2="45.085" y2="9.525" width="0.6096" layer="16"/>
+<wire x1="45.085" y1="9.525" x2="47.625" y2="9.525" width="0.6096" layer="16"/>
+<wire x1="26.67" y1="21.33" x2="26.67" y2="15.875" width="0.4064" layer="1"/>
+<wire x1="26.67" y1="15.875" x2="33.02" y2="9.525" width="0.4064" layer="1"/>
+<wire x1="40.005" y1="9.525" x2="33.02" y2="9.525" width="0.4064" layer="1"/>
 </signal>
 <signal name="D7">
@@
 <signal name="N$2">
 <contactref element="U$1" pad="16"/>
-<contactref element="LIGHT" pad="1"/>
-<wire x1="40.005" y1="9.525" x2="40.005" y2="10.795" width="0.4064" layer="1"/>
-<wire x1="40.005" y1="10.795" x2="39.37" y2="11.43" width="0.4064" layer="1"/>
-<wire x1="39.37" y1="11.43" x2="39.37" y2="17.52" width="0.4064" layer="1"/>
-<wire x1="39.37" y1="17.52" x2="35.56" y2="21.33" width="0.4064" layer="1"/>
+<contactref element="LIGHT" pad="8"/>
+<wire x1="35.56" y1="21.33" x2="35.56" y2="20.32" width="0.4064" layer="1"/>
+<wire x1="35.56" y1="20.32" x2="36.83" y2="19.05" width="0.4064" layer="1"/>
+<wire x1="36.83" y1="19.05" x2="43.18" y2="19.05" width="0.4064" layer="1"/>
+<wire x1="48.895" y1="12.065" x2="48.895" y2="13.335" width="0.4064" layer="1"/>
+<wire x1="48.895" y1="13.335" x2="43.18" y2="19.05" width="0.4064" layer="1"/>
 </signal>
 <signal name="N$3">
 <contactref element="U$1" pad="15"/>
-<contactref element="LIGHT" pad="3"/>
-<wire x1="42.545" y1="9.525" x2="42.545" y2="8.255" width="0.4064" layer="1"/>
-<wire x1="42.545" y1="8.255" x2="41.91" y2="7.62" width="0.4064" layer="1"/>
-<wire x1="41.91" y1="7.62" x2="38.1" y2="7.62" width="0.4064" layer="1"/>
-<wire x1="38.1" y1="7.62" x2="34.29" y2="11.43" width="0.4064" layer="1"/>
-<wire x1="34.29" y1="11.43" x2="34.29" y2="21.33" width="0.4064" layer="1"/>
+<contactref element="LIGHT" pad="6"/>
+<wire x1="46.355" y1="12.065" x2="46.355" y2="13.335" width="0.4064" layer="1"/>
+<wire x1="46.355" y1="13.335" x2="41.275" y2="18.415" width="0.4064" layer="1"/>
+<wire x1="41.275" y1="18.415" x2="36.195" y2="18.415" width="0.4064" layer="1"/>
+<wire x1="36.195" y1="18.415" x2="34.29" y2="20.32" width="0.4064" layer="1"/>
+<wire x1="34.29" y1="20.32" x2="34.29" y2="21.33" width="0.4064" layer="1"/>
+</signal>
+<signal name="N$5">
+<contactref element="U$1" pad="13"/>
+<contactref element="LIGHT" pad="2"/>
+<wire x1="41.275" y1="12.065" x2="41.275" y2="13.97" width="0.4064" layer="1"/>
+<wire x1="41.275" y1="13.97" x2="38.1" y2="17.145" width="0.4064" layer="1"/>
+<wire x1="38.1" y1="17.145" x2="34.925" y2="17.145" width="0.4064" layer="1"/>
+<wire x1="34.925" y1="17.145" x2="31.75" y2="20.32" width="0.4064" layer="1"/>
+<wire x1="31.75" y1="20.32" x2="31.75" y2="21.33" width="0.4064" layer="1"/>
 </signal>
 <signal name="N$4">
 <contactref element="U$1" pad="14"/>
-<contactref element="LIGHT" pad="5"/>
-<wire x1="33.02" y1="21.33" x2="33.02" y2="11.43" width="0.4064" layer="1"/>
-<wire x1="33.02" y1="11.43" x2="37.465" y2="6.985" width="0.4064" layer="1"/>
-<wire x1="37.465" y1="6.985" x2="44.45" y2="6.985" width="0.4064" layer="1"/>
-<wire x1="44.45" y1="6.985" x2="45.085" y2="7.62" width="0.4064" layer="1"/>
-<wire x1="45.085" y1="7.62" x2="45.085" y2="9.525" width="0.4064" layer="1"/>
-</signal>
-<signal name="N$5">
-<contactref element="LIGHT" pad="7"/>
-<contactref element="U$1" pad="13"/>
-<wire x1="47.625" y1="9.525" x2="47.625" y2="6.985" width="0.4064" layer="1"/>
-<wire x1="47.625" y1="6.985" x2="46.99" y2="6.35" width="0.4064" layer="1"/>
-<wire x1="46.99" y1="6.35" x2="36.83" y2="6.35" width="0.4064" layer="1"/>
-<wire x1="36.83" y1="6.35" x2="31.75" y2="11.43" width="0.4064" layer="1"/>
-<wire x1="31.75" y1="11.43" x2="31.75" y2="21.33" width="0.4064" layer="1"/>
+<contactref element="LIGHT" pad="4"/>
+<wire x1="33.02" y1="21.33" x2="33.02" y2="20.32" width="0.4064" layer="1"/>
+<wire x1="33.02" y1="20.32" x2="35.56" y2="17.78" width="0.4064" layer="1"/>
+<wire x1="35.56" y1="17.78" x2="39.37" y2="17.78" width="0.4064" layer="1"/>
+<wire x1="39.37" y1="17.78" x2="43.815" y2="13.335" width="0.4064" layer="1"/>
+<wire x1="43.815" y1="13.335" x2="43.815" y2="12.065" width="0.4064" layer="1"/>
 </signal>
 </signals>
